File: EINK_DEV/EINK_DEV_OLD_PCB.kicad_pcb (KiCad board)
At the start: 2 copper layers, 50.5 x 46.5 mm, 76 parts, among them J1 FPC, J2 Conn_01x06, J3 Conn_01x02, J4 Conn_01x03, J5 Conn_ARM_SWD_TagConnect_TC2030, J6 UART, J7 Conn_Coaxial, J8 GPIO_Header_Dev, P1 USB_C_Plug_USB2.0, Q1 Si1304BDL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

Commit message: PCB
Parts:
- R14: moved to B.Cu
- moved Y2 27.9 mm to (151.6, 112.6), turned to 0 degrees
- moved C24 27.5 mm to (154.5, 79.3), turned to -90 degrees
- moved C33 23.2 mm to (139.0, 89.7), turned to 90 degrees
- moved R14 17.3 mm to (145.5, 95.5)
- moved C17 16.6 mm to (142.0, 93.2), turned to -90 degrees
- moved C18 16.1 mm to (139.0, 93.3), turned to -90 degrees
- moved R9 15.5 mm to (175.0, 88.7), turned to 90 degrees
- moved J5 10.3 mm to (139.9, 105.0)
- moved C27 9.85 mm to (142.0, 96.8), turned to 90 degrees
- moved C26 9.32 mm to (139.0, 96.7), turned to 90 degrees
- moved R4 8.27 mm to (167.3, 78.5)
- moved D4 7.98 mm to (167.4, 80.5)
- moved L4 5.39 mm to (154.2, 106.5)
- moved C28 5.38 mm to (151.8, 109.0)
- moved C21 4.96 mm to (153.5, 75.7), turned to -90 degrees
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Routing:
- net Net-(J5-SWCLK): track 0.00 -> 80.4 mm, vias 0 -> 2
- net D-: track 0.00 -> 66.5 mm, vias 0 -> 7
- net Net-(J4-Pin_3): track 15.4 -> 67.6 mm
- net D+: track 0.00 -> 50.8 mm, vias 0 -> 4
- net GND: track 274.2 -> 324.5 mm, vias 4 -> 5
- net VGL: track 5.08 -> 54.3 mm, vias 0 -> 4
- net Net-(J8-Pin_3): track 2.08 -> 43.2 mm, vias 0 -> 2
- net Net-(J8-Pin_2): track 0.00 -> 32.4 mm, vias 0 -> 1
- net Net-(D4-A): track 30.4 -> 61.7 mm, vias 0 -> 6
- net Net-(J2-Pin_1): track 0.00 -> 30.5 mm
- net Net-(J8-Pin_9): track 0.00 -> 28.6 mm
- net Net-(J2-Pin_4): track 14.8 -> 43.2 mm
- net RESE: track 59.9 -> 34.3 mm
- net Net-(U1-PA3): track 0.00 -> 25.4 mm, vias 0 -> 3
- net Net-(U1-OSC_OUT): track 6.59 -> 31.1 mm, vias 0 -> 2
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