File: EINK_DEV/EINK_DEV.kicad_sch (KiCad schematic)
At the start: 75 parts, among them J1 FPC, J3 Conn_01x02, J4 Conn_01x03, J5 Conn_ARM_SWD_TagConnect_TC2030, J6 UART, J7 Conn_Coaxial, J8 GPIO_Header_Dev, P1 USB_C_Plug_USB2.0, Q1 NMOS, SW1 SW_Push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

Commit message: SPI conn, bigger sheet, rf mod replace
Parts:
- added U4: STM32WB5MMGH6TR, STM32WB5MMGH6TR:XCVR_STM32WB5MMGH6TR, symbol STM32WB5MMGH6TR:STM32WB5MMGH6TR
- U1: value STM32WB55CEUx -> STM32WB55CEU6
Connections:
- net CS# is gone; now on net CS#_SCREEN: J1.12 (Pin_12)
- net SCL is gone; now on net SCL_SCREEN: J1.13 (Pin_13)
- net SCL_SCREEN: now reaches R12.2, U1.11 (PA2)
- net SCL_SCREEN: now also R13.2, U1.10 (PA1), U1.12 (PA3)
- net at D6.2 (A): now also U1.17 (PA8); no longer U1.16 (PA7)
- net CS#_SCREEN: now reaches U1.15 (PA6)
- net SDA renamed SDA_SCREEN
- net SDA_SCREEN: now also U1.16 (PA7)
Other:
- note added: "STM32WB55CEU6 REQ. COMP"
- note added: "replacement STM32WB5MMGH6TR with intergrated 2,4 GHz Antenna"
- moved on the sheet: C1, C10, C11, C12, C14, C15, C16, C17, C18, C19, C2, C20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

Commit message: Dużo zmian ale to jeszcze nie koniec
Parts:
- removed U4: STM32WB5MMGH6TR, STM32WB5MMGH6TR:XCVR_STM32WB5MMGH6TR, symbol STM32WB5MMGH6TR:STM32WB5MMGH6TR
- added J2: Conn_01x06, Connector_Molex:Molex_KK-254_AE-6410-06A_1x06_P2.54mm_Vertical, symbol Connector_Generic:Conn_01x06
- C1, C10, C2, C5, C7, C8, C9: value C_Small -> 1u; footprint (none) -> Capacitor_SMD:C_0603_1608Metric
- C11, C12, C14, C15, C16, C17, C18, C19, C20, C21, C22, C23, C24, C25, C26, C27, C28, C29, C30, C31, C32, C33: footprint (none) -> Capacitor_SMD:C_0603_1608Metric
- C3, C6: value C_Small -> 1uF; footprint (none) -> Capacitor_SMD:C_0603_1608Metric
- C4: value C_Small -> uF; footprint (none) -> Capacitor_SMD:C_0603_1608Metric
- D1, D2, D3: footprint (none) -> Diode_SMD:D_0603_1608Metric
- D4, D5, D6: footprint (none) -> LED_SMD:LED_0603_1608Metric
- J1: footprint (none) -> Connector_FFC-FPC:TE_2-1734839-4_1x24-1MP_P0.5mm_Horizontal
- J3: footprint (none) -> Connector_Molex:Molex_KK-254_AE-6410-02A_1x02_P2.54mm_Vertical
- J4: footprint (none) -> Connector:FanPinHeader_1x03_P2.54mm_Vertical
- J6: footprint (none) -> Connector:FanPinHeader_1x04_P2.54mm_Vertical
- J7: footprint (none) -> Connector_Coaxial:U.FL_Hirose_U.FL-R-SMT-1_Vertical
- J8: footprint (none) -> Connector_Harwin:Harwin_M20-89010xx_1x10_P2.54mm_Horizontal
- JP1: footprint (none) -> Connector_PinHeader_2.54mm:PinHeader_1x03_P2.54mm_Horizontal
- L1, L2, L3, L4: footprint (none) -> Inductor_SMD:L_0603_1608Metric
- P1: footprint (none) -> Connector_USB:USB_C_Plug_Molex_105444
- Q1: value NMOS -> Si1304BDL; footprint (none) -> footprints:SC-70_SI1_VIS
- R1, R10, R11, R2, R3, R4, R5, R6, R7, R8, R9, TH1: footprint (none) -> Resistor_SMD:R_0603_1608Metric
- R12, R13, R15: value 220R -> 220; footprint (none) -> Resistor_SMD:R_0603_1608Metric
- R14: value 5k1 -> 5100; footprint (none) -> Resistor_SMD:R_0603_1608Metric
- SW1: footprint (none) -> Button_Switch_THT:SW_PUSH_6mm
- Y1: footprint (none) -> Crystal:Crystal_SMD_2012-2Pin_2.0x1.2mm
- Y2: footprint (none) -> Crystal:Crystal_SMD_2016-4Pin_2.0x1.6mm
Connections:
- net OUT+ is gone; now on net VBUS: C12.2, C31.1, JP1.2 (C), U2.5 (BAT), U3.1 (EN), U3.2 (IN)
- net VCC is gone; now on net +3V3: C1.1, L1.1, R2.1
- net +3.3V: no longer C23.1, J5.1 (VCC), U1.23 (VDDRF)
- net +3V3: now also C23.1, J5.1 (VCC), U1.23 (VDDRF)
- net SCL_SCREEN: no longer R12.2, R13.2, U1.11 (PA2), U1.12 (PA3)
- net at U1.13 (PA4): now also J2.2 (Pin_2)
- net at U1.14 (PA5): now also J2.3 (Pin_3)
- net at U1.18 (PA9): now also J2.4 (Pin_4)
- net at U1.36 (PA10): now also J2.5 (Pin_5)
- net at U1.42 (PA15): now also J2.6 (Pin_6)
- net at U1.9 (PA0): now also J2.1 (Pin_1)
- new net: R12.2, U1.11 (PA2)
- new net: R13.2, U1.12 (PA3)
- no-connect marks 6 -> 11
Other:
- note added: "MOUNTING POINTS"
- note removed: "replacement STM32WB5MMGH6TR with intergrated 2,4 GHz Antenna"
- moved on the sheet: C1, C10, C11, C12, C14, C15, C16, C17, C18, C19, C2, C20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

Commit message: PCB
Parts:
- J2: footprint Connector_Molex:Molex_KK-254_AE-6410-06A_1x06_P2.54mm_Vertical -> Connector_PinHeader_2.54mm:PinHeader_1x06_P2.54mm_Horizontal
- J6: footprint Connector:FanPinHeader_1x04_P2.54mm_Vertical -> Connector_PinHeader_2.54mm:PinHeader_1x04_P2.54mm_Horizontal
- J8: footprint Connector_Harwin:Harwin_M20-89010xx_1x10_P2.54mm_Horizontal -> Connector_PinHeader_2.54mm:PinHeader_1x10_P2.54mm_Horizontal
Changed lines of the file:
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@@
 			)
 		)
-		(property "Footprint" "Connector:FanPinHeader_1x04_P2.54mm_Vertical"
+		(property "Footprint" "Connector_PinHeader_2.54mm:PinHeader_1x04_P2.54mm_Horizontal"
 			(at 39.37 67.31 0)
 			(effects
@@
 			)
 		)
-		(property "Footprint" "Connector_Molex:Molex_KK-254_AE-6410-06A_1x06_P2.54mm_Vertical"
+		(property "Footprint" "Connector_PinHeader_2.54mm:PinHeader_1x06_P2.54mm_Horizontal"
 			(at 54.61 97.79 0)
 			(effects
@@
 			)
 		)
-		(property "Footprint" "Connector_Harwin:Harwin_M20-89010xx_1x10_P2.54mm_Horizontal"
+		(property "Footprint" "Connector_PinHeader_2.54mm:PinHeader_1x10_P2.54mm_Horizontal"
 			(at 68.58 130.81 0)
 			(effects

Commit message: PCB gotowa
Parts:
- removed J2: Conn_01x06, Connector_PinHeader_2.54mm:PinHeader_1x06_P2.54mm_Horizontal, symbol Connector_Generic:Conn_01x06
- added J2: UART1, Connector_PinHeader_2.54mm:PinHeader_1x04_P2.54mm_Horizontal, symbol Connector_Generic:Conn_01x04
- added J9: USER2, Connector_PinHeader_2.54mm:PinHeader_1x04_P2.54mm_Horizontal, symbol Connector_Generic:Conn_01x04
- J6: value UART -> LOW POWER UART
- J8: value GPIO_Header_Dev -> USER1
Connections:
- net +3.3V: now also J2.1 (Pin_1)
- net GND: now also J2.4 (Pin_4)
- net at U1.13 (PA4): now also J9.2 (Pin_2)
- net at U1.14 (PA5): now also J9.3 (Pin_3)
- net at U1.18 (PA9): now also J2.2 (Pin_2)
- net at U1.36 (PA10): now also J2.3 (Pin_3)
- net at U1.42 (PA15): now also J9.4 (Pin_4)
- net at U1.9 (PA0): now also J9.1 (Pin_1)
